File: muricoca.kicad_pcb (KiCad board)
At the start: 2 copper layers, 24 parts, among them J1 USB_B_Mini, SW1 MXSwitch, SW2 MXSwitch, SW3 MXSwitch, SW4 MXSwitch, U1 ATmega32U4-AU, Y1 16Mhz

Commit message: feat: align the switches on the PCB
Parts:
- added D10: 1N4148W, Diode_SMD:D_SOD-123, F.Cu at (261.6, 201.6)
- added D11: 1N4148W, Diode_SMD:D_SOD-123, F.Cu at (255.9, 201.6)
- added D12: 1N4148W, Diode_SMD:D_SOD-123, F.Cu at (250.1, 201.6)
- added D13: 1N4148W, Diode_SMD:D_SOD-123, F.Cu at (244.4, 201.6)
- added D14: 1N4148W, Diode_SMD:D_SOD-123, F.Cu at (238.6, 201.6)
- added D15: 1N4148W, Diode_SMD:D_SOD-123, F.Cu at (232.9, 201.6)
- added D16: 1N4148W, Diode_SMD:D_SOD-123, F.Cu at (227.1, 201.6)
- added D17: 1N4148W, Diode_SMD:D_SOD-123, F.Cu at (221.4, 201.6)
- added D18: 1N4148W, Diode_SMD:D_SOD-123, F.Cu at (267.4, 201.6)
- added D19: 1N4148W, Diode_SMD:D_SOD-123, F.Cu at (209.9, 201.6)
- added D20: 1N4148W, Diode_SMD:D_SOD-123, F.Cu at (204.1, 201.6)
- added D21: 1N4148W, Diode_SMD:D_SOD-123, F.Cu at (198.4, 201.6)
- added D22: 1N4148W, Diode_SMD:D_SOD-123, F.Cu at (192.6, 201.6)
- added D23: 1N4148W, Diode_SMD:D_SOD-123, F.Cu at (186.9, 201.6)
- added D24: 1N4148W, Diode_SMD:D_SOD-123, F.Cu at (273.1, 201.6)
- added D25: 1N4148W, Diode_SMD:D_SOD-123, F.Cu at (181.1, 201.6)
- added D26: 1N4148W, Diode_SMD:D_SOD-123, F.Cu at (175.4, 201.6)
- added D27: 1N4148W, Diode_SMD:D_SOD-123, F.Cu at (278.9, 201.6)
- added D28: 1N4148W, Diode_SMD:D_SOD-123, F.Cu at (140.9, 198.3)
- added D29: 1N4148W, Diode_SMD:D_SOD-123, F.Cu at (146.6, 198.3)
- added D30: 1N4148W, Diode_SMD:D_SOD-123, F.Cu at (152.4, 198.3)
- added D31: 1N4148W, Diode_SMD:D_SOD-123, F.Cu at (158.1, 198.3)
- added D32: 1N4148W, Diode_SMD:D_SOD-123, F.Cu at (163.9, 198.3)
- added D33: 1N4148W, Diode_SMD:D_SOD-123, F.Cu at (169.6, 198.3)
- added D34: 1N4148W, Diode_SMD:D_SOD-123, F.Cu at (175.4, 198.3)
- added D35: 1N4148W, Diode_SMD:D_SOD-123, F.Cu at (181.1, 198.3)
- added D36: 1N4148W, Diode_SMD:D_SOD-123, F.Cu at (186.9, 198.3)
- added D37: 1N4148W, Diode_SMD:D_SOD-123, F.Cu at (192.6, 198.3)
- added D38: 1N4148W, Diode_SMD:D_SOD-123, F.Cu at (198.4, 198.3)
- added D39: 1N4148W, Diode_SMD:D_SOD-123, F.Cu at (204.1, 198.3)
- added D40: 1N4148W, Diode_SMD:D_SOD-123, F.Cu at (209.9, 198.3)
- added D41: 1N4148W, Diode_SMD:D_SOD-123, F.Cu at (215.6, 198.3)
- added D42: 1N4148W, Diode_SMD:D_SOD-123, F.Cu at (278.9, 198.3)
- added D43: 1N4148W, Diode_SMD:D_SOD-123, F.Cu at (232.9, 198.3)
- added D44: 1N4148W, Diode_SMD:D_SOD-123, F.Cu at (238.6, 198.3)
- added D45: 1N4148W, Diode_SMD:D_SOD-123, F.Cu at (244.4, 198.3)
- added D46: 1N4148W, Diode_SMD:D_SOD-123, F.Cu at (250.1, 198.3)
- added D47: 1N4148W, Diode_SMD:D_SOD-123, F.Cu at (255.9, 198.3)
- added D48: 1N4148W, Diode_SMD:D_SOD-123, F.Cu at (261.6, 198.3)
- added D49: 1N4148W, Diode_SMD:D_SOD-123, F.Cu at (267.4, 198.3)
- added D5: 1N4148W, Diode_SMD:D_SOD-123, F.Cu at (152.4, 201.6)
- added D50: 1N4148W, Diode_SMD:D_SOD-123, F.Cu at (273.1, 198.3)
- added D51: 1N4148W, Diode_SMD:D_SOD-123, F.Cu at (227.1, 198.3)
- added D52: 1N4148W, Diode_SMD:D_SOD-123, F.Cu at (284.6, 198.7)
- added D53: 1N4148W, Diode_SMD:D_SOD-123, F.Cu at (284.6, 195.3)
- added D54: 1N4148W, Diode_SMD:D_SOD-123, F.Cu at (284.6, 192.0)
- added D55: 1N4148W, Diode_SMD:D_SOD-123, F.Cu at (284.6, 188.6)
- added D56: 1N4148W, Diode_SMD:D_SOD-123, F.Cu at (284.6, 185.3)
- added D57: 1N4148W, Diode_SMD:D_SOD-123, F.Cu at (283.4, 181.9)
- added D58: 1N4148W, Diode_SMD:D_SOD-123, F.Cu at (221.4, 198.3)
- added D6: 1N4148W, Diode_SMD:D_SOD-123, F.Cu at (158.1, 201.6)
- added D7: 1N4148W, Diode_SMD:D_SOD-123, F.Cu at (163.9, 201.6)
- added D8: 1N4148W, Diode_SMD:D_SOD-123, F.Cu at (169.6, 201.6)
- added D9: 1N4148W, Diode_SMD:D_SOD-123, F.Cu at (215.6, 201.6)
- added R5: 330R, Resistor_SMD:R_1206_3216Metric_Pad1.42x1.75mm_HandSolder, F.Cu at (289.2, 202.1)
- added SW10: 9, acheron_MX:MX100, B.Cu at (188.1, -104.8)
- added SW11: 0, acheron_MX:MX100, B.Cu at (207.2, -104.8)
- added SW12: -, acheron_MX:MX100, B.Cu at (226.2, -104.8)
- added SW13: =, acheron_MX:MX100, B.Cu at (245.3, -104.8)
- added SW14: Bksp_200, acheron_MX:MX200, B.Cu at (273.8, -104.8)
- added SW15: Tab_150, acheron_MX:MX150, B.Cu at (21.4, -85.7)
- added SW16: Q, acheron_MX:MX100, B.Cu at (45.2, -85.7)
- added SW17: W, acheron_MX:MX100, B.Cu at (64.3, -85.7)
- added SW18: E, acheron_MX:MX100, B.Cu at (83.3, -85.7)
- added SW19: R, acheron_MX:MX100, B.Cu at (102.4, -85.7)
- added SW20: T, acheron_MX:MX100, B.Cu at (121.4, -85.7)
- added SW21: Y, acheron_MX:MX100, B.Cu at (140.5, -85.7)
- added SW22: U, acheron_MX:MX100, B.Cu at (159.5, -85.7)
- added SW23: I, acheron_MX:MX100, B.Cu at (178.6, -85.7)
- added SW24: O, acheron_MX:MX100, B.Cu at (197.6, -85.7)
- added SW25: P, acheron_MX:MX100, B.Cu at (216.7, -85.7)
- added SW26: [, acheron_MX:MX100, B.Cu at (235.7, -85.7)
- added SW27: ], acheron_MX:MX100, B.Cu at (254.8, -85.7)
- added SW28: \_150, acheron_MX:MX150, B.Cu at (278.6, -85.7)
- added SW29: Caps_175, acheron_MX:MX175, B.Cu at (23.8, -66.7)
- added SW30: A, acheron_MX:MX100, B.Cu at (50.0, -66.7)
- added SW31: S, acheron_MX:MX100, B.Cu at (69.1, -66.7)
- added SW32: D, acheron_MX:MX100, B.Cu at (88.1, -66.7)
- added SW33: F, acheron_MX:MX100, B.Cu at (107.2, -66.7)
- added SW34: G, acheron_MX:MX100, B.Cu at (126.2, -66.7)
- added SW35: H, acheron_MX:MX100, B.Cu at (145.3, -66.7)
- added SW36: J, acheron_MX:MX100, B.Cu at (164.3, -66.7)
- added SW37: K, acheron_MX:MX100, B.Cu at (183.4, -66.7)
- added SW38: L, acheron_MX:MX100, B.Cu at (202.4, -66.7)
- added SW39: ;, acheron_MX:MX100, B.Cu at (221.5, -66.7)
- added SW40: ', acheron_MX:MX100, B.Cu at (240.5, -66.7)
- added SW41: Enter_225, acheron_MX:MX225, B.Cu at (271.5, -66.7)
- added SW42: LShift_225, acheron_MX:MX225, B.Cu at (28.6, -47.6)
- added SW43: Z, acheron_MX:MX100, B.Cu at (59.5, -47.6)
- added SW44: X, acheron_MX:MX100, B.Cu at (78.6, -47.6)
- added SW45: C, acheron_MX:MX100, B.Cu at (97.6, -47.6)
- added SW46: V, acheron_MX:MX100, B.Cu at (116.7, -47.6)
- added SW47: B, acheron_MX:MX100, B.Cu at (135.7, -47.6)
- added SW48: N, acheron_MX:MX100, B.Cu at (154.8, -47.6)
- added SW49: M, acheron_MX:MX100, B.Cu at (173.8, -47.6)
- added SW5: 4, acheron_MX:MX100, B.Cu at (92.9, -104.8)
- added SW50: ,, acheron_MX:MX100, B.Cu at (192.9, -47.6)
- added SW51: ., acheron_MX:MX100, B.Cu at (211.9, -47.6)
- added SW52: /, acheron_MX:MX100, B.Cu at (231.0, -47.6)
- added SW53: RShift_275, acheron_MX:MX275, B.Cu at (266.7, -47.6)
- added SW54: LCtrl_150, acheron_MX:MX150, B.Cu at (21.4, -28.6)
- added SW55: Alt_150, acheron_MX:MX150, B.Cu at (69.1, -28.6)
- added SW56: Space_700, acheron_MX:MX700, B.Cu at (150.0, -28.6)
- added SW57: Alt Gr_150, acheron_MX:MX150, B.Cu at (231.0, -28.6)
- added SW58: RCtrl_150, acheron_MX:MX150, B.Cu at (278.6, -28.6)
- added SW6: 5, acheron_MX:MX100, B.Cu at (111.9, -104.8)
- added SW7: 6, acheron_MX:MX100, B.Cu at (131.0, -104.8)
- added SW8: 7, acheron_MX:MX100, B.Cu at (150.0, -104.8)
- added SW9: 8, acheron_MX:MX100, B.Cu at (169.1, -104.8)
- D1, D2, D3, D4: value D_Small -> 1N4148W
- R4: value 10k -> 1k
- SW1: value MXSwitch -> Esc; moved to B.Cu
- SW2: value MXSwitch -> 1; moved to B.Cu
- SW3: value MXSwitch -> 2; moved to B.Cu
- SW4: value MXSwitch -> 3; moved to B.Cu
- moved SW1 240.4 mm to (16.7, -104.8), turned to 180 degrees
- moved SW3 219.5 mm to (54.8, -104.8), turned to 180 degrees
- moved SWP1 216.9 mm to (331.8, 204.2), turned to 180 degrees
- moved R2 216.5 mm to (301.1, 202.1), turned to 180 degrees
- moved SW2 213.8 mm to (35.7, -104.8), turned to 180 degrees
- moved R3 211.0 mm to (307.1, 202.1), turned to 180 degrees
- moved R4 211.0 mm to (313.0, 202.1), turned to 180 degrees
- moved R1 205.5 mm to (295.2, 202.1), turned to 180 degrees
- moved Y1 196.3 mm to (321.1, 202.8), turned to 180 degrees
- moved SW4 195.9 mm to (73.8, -104.8), turned to 180 degrees
- moved D3 175.9 mm to (283.4, 205.0), turned to 180 degrees
- moved D2 169.2 mm to (277.6, 205.0), turned to 180 degrees
- moved D1 162.9 mm to (271.9, 205.0), turned to 180 degrees
- moved C3 157.3 mm to (266.6, 204.8), turned to 180 degrees
- moved C4 155.0 mm to (261.9, 204.8), turned to 180 degrees
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Connections:
- C1 pad 2: GND -> Net-(C1-Pad2)
- D3 pad 1: ROW2 -> ROW1
- D4 pad 1: ROW2 -> ROW1
- SW3 pad 1: COL1 -> COL3
- SW4 pad 1: COL2 -> COL4
- SWP1 pad 1: GND -> Net-(C1-Pad2)
